File: LCD_connectors.kicad_sch (KiCad schematic)
At the start: 2 parts, among them J4 LCD SPI, J4 LCD Soft SPI

Commit message: Rev 0.3: Passage sur deux couches
Passage sur deux couches, ajustement de l'impédance pour l'USB.
Reroutage de l'alimentation côté USB
Ajout de beaucoup de silk
Quelques ajustements de nets pour la lisbilité
Ajout de LEDs de debug
Plan de masse sur le top
Quelques mises à jour sur le schematic
Parts:
- J4: now left out of the parts list
Changed lines of the file:
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@@
   (title_block
     (title "Projet Barbapapa")
-    (date "2023-06-22")
-    (rev "0.2")
+    (date "2023-06-25")
+    (rev "0.3")
     (company "Téo-CD")
   )
@@
   )
   (symbol (lib_id "Connector_Generic:Conn_02x04_Top_Bottom") (at 104.14 54.61 0) (unit 1)
-    (in_bom yes) (on_board yes) (dnp no) (fields_autoplaced)
+    (in_bom no) (on_board yes) (dnp no) (fields_autoplaced)
     (property "Reference" "J4" (at 105.41 45.72 0)
       (effects (font (size 1.27 1.27)))
@@
   )
   (symbol (lib_id "Connector_Generic:Conn_02x04_Top_Bottom") (at 104.14 73.66 0) (unit 1)
-    (in_bom yes) (on_board yes) (dnp no) (fields_autoplaced)
+    (in_bom no) (on_board yes) (dnp no) (fields_autoplaced)
     (property "Reference" "J4" (at 105.41 64.77 0)
       (effects (font (size 1.27 1.27)))
