File: NFC_Connectors.kicad_sch (KiCad schematic)
At the start: 2 parts, among them J7 NFC1, J8 NFC2

Commit message: Rev 0.3: Passage sur deux couches
Passage sur deux couches, ajustement de l'impédance pour l'USB.
Reroutage de l'alimentation côté USB
Ajout de beaucoup de silk
Quelques ajustements de nets pour la lisbilité
Ajout de LEDs de debug
Plan de masse sur le top
Quelques mises à jour sur le schematic
Parts:
- J7, J8: now left out of the parts list
Changed lines of the file:
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@@
   (title_block
     (title "Projet Barbapapa")
-    (date "2023-06-22")
-    (rev "0.2")
+    (date "2023-06-25")
+    (rev "0.3")
     (company "Téo-CD")
   )
@@
   )
   (symbol (lib_id "Connector_Generic:Conn_01x07") (at 111.76 64.77 0) (mirror y) (unit 1)
-    (in_bom yes) (on_board yes) (dnp no)
+    (in_bom no) (on_board yes) (dnp no)
     (property "Reference" "J8" (at 109.22 63.5 0)
       (effects (font (size 1.27 1.27)) (justify left))
@@
   )
   (symbol (lib_id "Connector_Generic:Conn_01x05") (at 91.44 62.23 0) (unit 1)
-    (in_bom yes) (on_board yes) (dnp no) (fields_autoplaced)
+    (in_bom no) (on_board yes) (dnp no) (fields_autoplaced)
     (property "Reference" "J7" (at 93.98 60.96 0)
       (effects (font (size 1.27 1.27)) (justify left))
