File: Projet_Barbapapa.kicad_pcb (KiCad board)
At the start: 2 copper layers, 85.1 x 99.9 mm, 47 parts, among them J1 USB_C_Receptacle_USB2.0, J2 Speaker, J3 Conn_01x02, J4 LCD SPI, J5 LCD Soft SPI, J6 Random FTDI, J7 NFC1, J8 NFC2, J9 RGB_LED, SW2 Power switch, U1 MAX98357A/B, U2 AP61201Z6-7 buck, U3 MAX1811, U4 CD4051B

Commit message: Change le Qr pour archive.org
Parts:
- G***: moved to B.Cu
- turned G*** to 180 degrees
